File: PCB/PCB.kicad_sch (KiCad schematic)
At the start: 22 parts, among them J1 IEC_C14_Receptacle, M1 Fan_4pin, M2 Motor_Servo, SW1 SW_SPST, SW2 SW_Push SET, SW3 SW_Push Pos1, SW4 SW_Push Pos2, U1 XIAO-RP2040-DIP, U2 Meanwell ELG-150-54B AC Side, U3 PC817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

Commit message: uhh did stuff by the looks of it
Parts:
- added U7: ~, symbol specialbits:Meanwell_PSU_1_1
- U6: value Meanwell ELG-150-54B Other side -> Meanwell ELG-150-54B dim pins
Connections:
- net at U6.1 (Dim+): now also U3.3; no longer D1.2 (A)
- net at U6.2 (Dim-): now also U3.4; no longer D1.1 (K)
- new net: D1.1 (K), U7.2 (Vo-)
- new net: D1.2 (A), U7.1 (Vo+)
Other:
- note added: "(freewired)"
Changed lines of the file:
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@@
 		)
 	)
+	(text "(freewired)"
+		(exclude_from_sim no)
+		(at 69.342 112.014 0)
+		(effects
+			(font
+				(size 1.27 1.27)
+			)
+		)
+	)
 	(text "Fused input receptacle"
 		(exclude_from_sim no)
@@
 			)
 		)
-		(property "Value" "Meanwell ELG-150-54B Other side"
+		(property "Value" "Meanwell ELG-150-54B dim pins"
 			(at 55.245 101.6 0)
 			(effects
@@
 			)
 		)
-		(pin "3"
-		)
 		(pin "1"
 		)
 		(pin "2"
 		)
-		(pin "4"
-		)
 		(instances
 			(project ""
@@
 		(exclude_from_sim no)
 		(in_bom yes)
-		(on_board yes)
+		(on_board no)
 		(dnp no)
 		(fields_autoplaced yes)
@@
 					(unit 1)
 				)
+			)
+		)
+	)
+	(symbol
+		(lib_id "specialbits:Meanwell_PSU_1_1")
+		(at 58.42 100.33 0)
+		(unit 1)
+		(exclude_from_sim no)
+		(in_bom yes)
+		(on_board no)
+		(dnp no)
+		(fields_autoplaced yes)
+		(property "Reference" "U7"
+			(at 60.325 99.06 0)
+			(effects
+				(font
+					(size 1.27 1.27)
+				)
+			)
+		)
+		(property "Value" "~"
+			(at 60.325 101.6 0)
+			(effects
+				(font
+					(size 1.27 1.27)
+				)
+			)
+		)
+		(property "Footprint" ""
+			(at 58.42 100.33 0)
+			(effects
+				(font
+					(size 1.27 1.27)
+				)
+				(hide yes)
+			)
+		)
+		(property "Datasheet" ""
+			(at 58.42 100.33 0)
+			(effects
+				(font
+					(size 1.27 1.27)
+				)
+				(hide yes)
+			)
+		)
+		(property "Description" ""
+			(at 58.42 100.33 0)
+			(effects
+				(font
+					(size 1.27 1.27)
+				)
+				(hide yes)
+			)
+		)
+		(pin "2"
+		)
+		(pin "1"
+		)
+		(instances
+			(project ""
+				(path "/cb8a0eb9-023d-474b-952c-ea4eac5ee9fe"
+					(reference "U7")
+					(unit 1)
+				)

Commit message: add slight pcb changes
Parts:
- removed U5: SMU02L-12, SMU02L_12:SIP750W50P254L1160H1014Q4, symbol SMU02L-12:SMU02L-12
- added U8: SPU03L-12, SPU03L-12:SPU03L-12_MWU, symbol SPU03L-12:SPU03L-12
- R2: value 42Ω 0.12W -> 80-100Ω
Connections:
- net +5V: now also U8.1 (VIN+)
- net GND: now also U8.2 (VIN-)
- net at M1.1 (-): now also U8.5 (VOUT-)
- net at M1.2 (+): now also U8.7 (VOUT+)
Other:
- moved on the sheet: M1
Changed lines of the file:
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@@
-	(wire
-		(pts
-			(xy 148.59 41.91) (xy 148.59 44.45)
-		)
-		(stroke
-			(width 0)
-			(type default)
-		)
-	)
 	(wire
 		(pts
@@
 		(pts
 			(xy 99.06 66.04) (xy 156.21 66.04)
+		)
+		(stroke
+			(width 0)
+			(type default)
+		)
+	)
+	(wire
+		(pts
+			(xy 148.59 41.91) (xy 148.59 46.99)
 		)
 		(stroke
@@
 			)
 		)
-		(property "Value" "42Ω  0.12W"
+		(property "Value" "80-100Ω"
 			(at 93.98 116.8399 0)
 			(effects
@@
 	)
 	(symbol
+		(lib_id "SPU03L-12:SPU03L-12")
+		(at 107.95 46.99 0)
+		(unit 1)
+		(exclude_from_sim no)
+		(in_bom yes)
+		(on_board yes)
+		(dnp no)
+		(fields_autoplaced yes)
+		(property "Reference" "U8"
+			(at 128.27 36.83 0)
+			(effects
+				(font
+					(size 1.524 1.524)
+				)
+			)
+		)
+		(property "Value" "SPU03L-12"
+			(at 128.27 39.37 0)
+			(effects
+				(font
+					(size 1.524 1.524)
+				)
+			)
+		)
+		(property "Footprint" "SPU03L-12:SPU03L-12_MWU"
+			(at 107.95 46.99 0)
+			(effects
+				(font
+					(size 1.27 1.27)
+					(italic yes)
+				)
+				(hide yes)
+			)
+		)
+		(property "Datasheet" "SPU03L-05"
+			(at 107.95 46.99 0)
+			(effects
+				(font
+					(size 1.27 1.27)
+					(italic yes)
+				)
+				(hide yes)
+			)
+		)
+		(property "Description" ""
+			(at 107.95 46.99 0)
+			(effects
+				(font
+					(size 1.27 1.27)
+				)
+				(hide yes)
+			)
+		)
+		(pin "2"
+		)
+		(pin "1"
+		)
+		(pin "5"
+		)
+		(pin "7"
+		)
+		(instances
+			(project ""
+				(path "/cb8a0eb9-023d-474b-952c-ea4eac5ee9fe"
+					(reference "U8")
+					(unit 1)
+				)
+			)
+		)
+	)
+	(symbol
 		(lib_id "power:GND")
 		(at 83.82 120.65 90)
@@
 	(symbol
 		(lib_id "power:+5V")
-		(at 118.11 49.53 90)
-		(unit 1)
-		(exclude_from_sim no)
-		(in_bom yes)
-		(on_board yes)
-		(dnp no)
-		(fields_autoplaced yes)
+		(at 107.95 46.99 90)
+		(unit 1)
+		(exclude_from_sim no)
+		(in_bom yes)
+		(on_board yes)
+		(dnp no)
 		(property "Reference" "#PWR09"
-			(at 121.92 49.53 0)
+			(at 111.76 46.99 0)
 			(effects
 				(font
@@
 		)
 		(property "Value" "+5V"
-			(at 113.03 49.53 0)
+			(at 102.87 46.228 0)
 			(effects
 				(font
@@
 		)
 		(property "Footprint" ""
-			(at 118.11 49.53 0)
+			(at 107.95 46.99 0)
 			(effects
 				(font
@@
 		)
 		(property "Datasheet" ""
-			(at 118.11 49.53 0)
+			(at 107.95 46.99 0)
 			(effects
 				(font
@@
 		)
 		(property "Description" "Power symbol creates a global label with name \"+5V\""
-			(at 118.11 49.53 0)
+			(at 107.95 46.99 0)
 			(effects
 				(font
@@
 	(symbol
 		(lib_id "power:GND")
-		(at 118.11 44.45 270)
-		(unit 1)
-		(exclude_from_sim no)
-		(in_bom yes)
-		(on_board yes)
-		(dnp no)
-		(fields_autoplaced yes)
+		(at 107.95 49.53 270)
+		(unit 1)
+		(exclude_from_sim no)
+		(in_bom yes)
+		(on_board yes)
+		(dnp no)
 		(property "Reference" "#PWR08"
-			(at 111.76 44.45 0)
+			(at 101.6 49.53 0)
 			(effects
 				(font
@@
 		)
 		(property "Value" "GND"
-			(at 113.03 44.45 0)
+			(at 102.87 51.308 0)
 			(effects
 				(font
@@
 		)
 		(property "Footprint" ""
-			(at 118.11 44.45 0)
+			(at 107.95 49.53 0)
 			(effects
 				(font
@@
 		)
 		(property "Datasheet" ""
-			(at 118.11 44.45 0)
+			(at 107.95 49.53 0)
 			(effects
 				(font
@@
 		)
 		(property "Description" "Power symbol creates a global label with name \"GND\" , ground"
-			(at 118.11 44.45 0)
+			(at 107.95 49.53 0)
 			(effects
 				(font
@@
 	(symbol
 		(lib_id "Motor:Fan_4pin")
-		(at 165.1 46.99 180)
+		(at 165.1 49.53 0)
 		(unit 1)
 		(exclude_from_sim no)
@@
 		(fields_autoplaced yes)
 		(property "Reference" "M1"
-			(at 160.02 48.2601 0)
+			(at 170.18 48.2599 0)
 			(effects
 				(font
@@
 		)
 		(property "Value" "Fan_4pin"
-			(at 160.02 45.7201 0)
+			(at 170.18 50.7999 0)
 			(effects
 				(font
@@
 		)
 		(property "Footprint" "Connector:FanPinHeader_1x04_P2.54mm_Vertical"
-			(at 165.1 47.244 0)
+			(at 165.1 49.276 0)
 			(effects
 				(font
@@
 		)
 		(property "Datasheet" "http://www.formfactors.org/developer%5Cspecs%5Crev1_2_public.pdf"
-			(at 165.1 47.244 0)
+			(at 165.1 49.276 0)
 			(effects
 				(font
@@
 		)
 		(property "Description" "Fan, tacho output, PWM input, 4-pin connector"
-			(at 165.1 46.99 0)
+			(at 165.1 49.53 0)
 			(effects
 				(font
@@
 					(unit 1)
 				)
-			)
-		)
-	)
-	(symbol
-		(lib_id "SMU02L-12:SMU02L-12")
-		(at 133.35 46.99 0)
-		(unit 1)
-		(exclude_from_sim no)
-		(in_bom yes)
-		(on_board yes)
-		(dnp no)
-		(fields_autoplaced yes)
-		(property "Reference" "U5"
-			(at 133.35 36.83 0)
-			(effects
-				(font
-					(size 1.27 1.27)
-				)
-			)
-		)
-		(property "Value" "SMU02L-12"
-			(at 133.35 39.37 0)
-			(effects
-				(font
-					(size 1.27 1.27)
-				)
-			)
-		)
-		(property "Footprint" "SMU02L_12:SIP750W50P254L1160H1014Q4"
-			(at 133.35 46.99 0)
-			(effects
-				(font
-					(size 1.27 1.27)
-				)
-				(justify bottom)
-				(hide yes)
-			)
-		)
-		(property "Datasheet" ""
-			(at 133.35 46.99 0)
-			(effects
-				(font
-					(size 1.27 1.27)
-				)
-				(hide yes)
-			)
-		)
-		(property "Description" ""
-			(at 133.35 46.99 0)
-			(effects
-				(font
-					(size 1.27 1.27)
-				)
-				(hide yes)
-			)
-		)
-		(property "MF" "Mean Well"
-			(at 133.35 46.99 0)
-			(effects
-				(font
-					(size 1.27 1.27)
-				)
-				(justify bottom)
-				(hide yes)
-			)
-		)
-		(property "Mouser-Purchase-URL" "https://snapeda.com/shop?store=Mouser&id=2765143"
-			(at 133.35 46.99 0)
-			(effects
-				(font
-					(size 1.27 1.27)
-				)
-				(justify bottom)
-				(hide yes)
-			)
-		)
-		(property "Description_1" "Isolated Module DC DC Converter 1 Output 5V 400mA 4.5V - 5.5V Input"
-			(at 133.35 46.99 0)
-			(effects
-				(font
-					(size 1.27 1.27)
-				)
-				(justify bottom)
-				(hide yes)
-			)
-		)
-		(property "Package" "SIP-4 Mean Well"
-			(at 133.35 46.99 0)
-			(effects
-				(font
-					(size 1.27 1.27)
-				)
-				(justify bottom)
-				(hide yes)
-			)
-		)
-		(property "Price" "None"
-			(at 133.35 46.99 0)
-			(effects
-				(font
-					(size 1.27 1.27)
-				)
-				(justify bottom)
-				(hide yes)
-			)
-		)
-		(property "MP" "SMU02L-12"
-			(at 133.35 46.99 0)
-			(effects
-				(font
-					(size 1.27 1.27)
-				)
-				(justify bottom)
-				(hide yes)
-			)
-		)
-		(property "DigiKey-Purchase-URL" "https://snapeda.com/shop?store=DigiKey&id=2765143"
-			(at 133.35 46.99 0)
-			(effects
-				(font
-					(size 1.27 1.27)
-				)
-				(justify bottom)
-				(hide yes)
-			)
-		)
-		(property "Availability" "Unavailable"
-			(at 133.35 46.99 0)
-			(effects
-				(font
-					(size 1.27 1.27)
-				)
-				(justify bottom)
-				(hide yes)
-			)
-		)
-		(pin "4"
-		)
-		(pin "3"
-		)
-		(pin "1"
-		)
-		(pin "2"
-		)
-		(instances
-			(project ""
-				(path "/cb8a0eb9-023d-474b-952c-ea4eac5ee9fe"
-					(reference "U5")
-					(unit 1)
-				)
